File: schematics/et312.sch (EAGLE design)
At the start: 9 parts, among them IC1 MEGA16-P, IC2 4066N

Commit message: Schematic update
Added screen, finished buttons
Parts:
- removed R1: 500KOHM, 50mW, Panasonic-Trimmer_Potentiometers:EVJC20F02A14-JC2
- removed RV1: (no value), SparkFun-Electromechanical:POT
- added S1, S3: SPST, adafruit:SPST
- added VR2: 500KOHM, 50mW, Panasonic-Trimmer_Potentiometers:EVJC20F02A14-JC2
- added VR3: (no value), SparkFun-Electromechanical:POT
- added X1: HD44780LCD-1602, adafruit:HD44780LCD-1602
Connections:
- new net N$10: 10WAY_RIBBON.9, VR2.3'
- new net N$11: 10WAY_RIBBON.8, VR3.S
- new net N$12: 10WAY_RIBBON.7, RV2.S
- new net N$13: 10WAY_RIBBON.10, VR2.3
- new net N$14: 10WAY_RIBBON.4, VR2.2'
- new net N$15: 10WAY_RIBBON.3, VR2.2
- new net N$5: IC2D.A, S3.S
- new net N$7: 10WAY_RIBBON1.1, IC2B.A
- new net N$8: 10WAY_RIBBON1.2, IC2A.A
- new net N$9: 10WAY_RIBBON1.6
- new net PC0: IC1.(SCL)PC0, IC2A.C, IC2B.C, IC2C.C, IC2D.C
- new net PC1: IC1.(SDA)PC1, X1.RW
- new net PC2: IC1.(TCK)PC2, X1.E
- new net PC3: IC1.(TMS)PC3, X1.RS
- new net PC4: IC1.(TDO)PC4, IC2D.B, X1.DB4
- new net PC5: IC1.(TDI)PC5, IC2C.B, X1.DB5
- new net PC6: IC1.(TOSC1)PC6, IC2B.B, X1.DB6
- new net PC7: IC1.(TOSC2)PC7, IC2A.B, X1.DB7
- new net VR4: 10WAY_RIBBON.5, RV2.E, VR3.E
- net N$1: now also 10WAY_RIBBON.6, RV2.A, S2.P, S4.P, VR2.1, VR2.1', VR3.A; no longer IC2A.C
- net N$2: now also 10WAY_RIBBON.2, S2.S; no longer IC2B.C
- net N$3: now also 10WAY_RIBBON.1, S4.S; no longer IC2D.C
- net N$4: now also IC2C.A, S1.S; no longer IC2C.C
Other:
- note added: "Down"
- note added: "Level A"
- note added: "Level B"
- note added: "Multi Adjust"
- note added: "OK"
- note added: "The screen used is a WH1602A"
