File: hardware/schematics/arduino_sheild.brd (EAGLE design)
At the start: 68.6 x 53.3 mm, 37 parts, among them IC3 LM358, Q1 IRL520N-H, Q2 IRL520N-H, Q3 IRF9Z24, Q4 IRL520N-H, Q5 IRL520N-H, Q6 IRF9Z24, X5 STEREOJACK, X6 STEREOJACK

Commit message: Schematics
WIP
Parts:
- removed T2, T3: (no value), Eagle_POWER_MAGNETICS_rev16b:WE-FB_EFD25_DIMENSION1
- added TR1, TR2: 42TL025, trafo-xicon:42TL
- moved Q2 139.8 mm to (22.9, 5.08), turned to 180 degrees
- moved Q1 136.3 mm to (34.3, 5.08), turned to 180 degrees
- moved C3 127.8 mm to (-67.3, 11.4)
- moved C2 116.4 mm to (-68.6, 26.7)
- moved Q4 104.6 mm to (59.7, 50.8)
- moved IC3 101.7 mm to (27.9, 24.1)
- moved Q6 101.1 mm to (25.4, 50.8)
- moved Q5 97.7 mm to (36.8, 50.8)
- moved U$3 82.5 mm to (1.27, 1.27)
- moved X5 82.5 mm to (69.8, 27.9)
- moved X6 82.5 mm to (69.8, 12.7)
- moved Q3 81.0 mm to (48.3, 50.8)
Connections:
- removed net N$66: T3.11, X6.1
- removed net N$67: T3.8, X6.2, X6.5
- removed net N$77: T2.11, X5.1
- removed net N$78: T2.8, X5.2, X5.5
- new net N$1: TR1.4, X5.1
- new net N$2: TR1.6, X5.2, X5.5
- new net N$3: TR2.6, X6.2, X6.5
- new net N$4: TR2.4, X6.1
- net N$34: now also TR1.1; no longer T2.1
- net N$35: now also TR1.2; no longer T2.5
- net N$36: now also TR2.1; no longer T3.1
- net N$37: now also TR2.2; no longer T3.5
- net N$38: now also TR2.3; no longer T3.3
- net N$39: now also TR1.3; no longer T2.3
