File: hardware/schematics/arduino_shield.sch (EAGLE design)
At the start: 43 parts, among them IC1 LM358KIT, IC2 MAX548, Q1 IRL520N-H, Q2 IRF9Z24, Q3 IRL520N-H, Q4 IRL520N-H, Q5 IRF9Z24, Q6 IRL520N-H

Commit message: A Lot of work done :D
Assuming the Transformer is correct, we have a version we can send to a fab house
Parts:
- added C5, C9: 10uF, rcl:C-EUC0805K
- added C6, C8: 100nF, rcl:C-EUC0805K
- added C7: 47uF, rcl:CPOL-EUE2.5-5
- added LED1, LED2: (no value), adafruit:LEDCHIP-LED0805
- added R100: 0R, eagle-ltspice:R
- added R27, R28, R29: 100k, eagle-ltspice:R
- added R30: 560R, rcl:R-EU_R0805
- C1, C3: value 100nF -> 47uF; device capacitor-wima:C2.5/2 -> rcl:CPOL-EUE2.5-5
- R1: value 100k -> 1R
- R10: value 200k -> 100k
- R11, R19, R21, R22, R8: value 100k -> 10k
- R13, R15, R3, R5: value 10k -> 100k
- R14: value 10k -> xk
- R16, R4: value 100k -> 200k
- R2: value 10k -> 1R
- R20: value 200k -> 10k
- R23, R24: value 1R -> 10k
- R25: value 0R -> 100k
- R26: value 10k -> 560R; device eagle-ltspice:R -> rcl:R-EU_R0805
- R6: value 100k -> xk
Connections:
- new net N$7: IC2.!LDAC, R23.1
- new net N$8: LED1.A, R26.1
- new net N$9: LED2.A, R30.1
- net +12V: now also C1.+, C3.+, C4.2, C5.1, C6.1, C7.+, R12.2, R7.2; no longer C1.2, C4.1, R18.2, R8.2
- net +5V: now also C8.1, C9.1, R17.2, R23.2, R24.2, R3.2, R30.2; no longer C3.1, IC2.!LDAC, R19.2, R26.2, R9.2
- net ADC1: now also R1.2, R2.2; no longer R23.2, R24.2
- net GND: now also C1.-, C3.-, C5.2, C6.2, C7.-, C8.2, C9.2, LED1.C, LED2.C, R100.1, R15.1, R16.1, R2.1, R27.1, R28.1, R29.1, R9.1; no longer C3.2, C4.2, R10.1, R12.1, R17.1, R20.1, R21.1, R23.1, R24.1, R7.1
- net N$18: now also Q3.G, R20.2; no longer Q1.G, R2.2
- net N$19: now also Q1.G, R19.2; no longer Q3.G, R3.2
- net N$20: now also R10.2, R8.1; no longer R5.1, R6.2
- net N$21: now also C2.1, R8.2; no longer C1.1, R5.2
- net N$22: now also R5.2, R7.1, R9.2; no longer R11.2, R7.2, R8.1
- net N$24: now also Q6.G, R21.2; no longer Q4.G, R13.2
- net N$25: now also Q4.G, R22.2; no longer Q6.G, R14.2
- net N$26: now also R11.1, R13.2; no longer R15.1, R16.2
- net N$27: now also C4.1, R11.2; no longer C2.1, R15.2
- net N$28: now also R12.1, R15.2, R18.2; no longer R17.2, R18.1, R22.2
- net N$34: now also Q3.D; no longer Q1.D
- net N$35: now also R6.2
- net N$36: now also Q6.D; no longer Q4.D
- net N$37: now also R14.2
- net N$38: now also Q4.D; no longer Q6.D
- net N$39: now also Q1.D; no longer Q3.D
- net N$40: now also R10.1, R3.1, R4.2; no longer R10.2, R9.1
- net N$41: now also R13.1, R14.1, R16.2, R17.1; no longer R16.1, R19.1, R20.2
- net N$5: now also R5.1; no longer R11.1
- net N$6: now also R18.1; no longer R22.1
- net PIN2: now also R26.2
- net PIN3: now also R20.1, R25.2; no longer R1.2, R2.1
- net PIN4: now also R24.1; no longer R26.1
- net PIN5: now also R19.1, R27.2; no longer R14.1, R21.2
- net PIN6: now also R22.1, R29.2; no longer R3.1, R4.2
- net PIN9: now also R21.1, R28.2; no longer R12.2, R13.1
- net SHIELD: now also R100.2; no longer R25.2
